Commit message: Add missing head visuals to go2_x5 URDFs

File: source/robot_lab/data/Robots/go2_x5/go2_x5.mujoco.urdf (robot description, URDF)
Before this commit: robot go2_x5, 50 links, 49 joints
Links:
- link Head_lower: geometry collision sphere radius=0.047; visual sphere radius=0.047
- link Head_upper: geometry collision cylinder length=0.09 radius=0.05; visual cylinder length=0.09 radius=0.05

File: source/robot_lab/data/Robots/go2_x5/go2_x5.urdf (robot description, URDF)
Before this commit: robot go2_x5, 52 links, 51 joints
Links:
- link Head_lower: geometry collision sphere radius=0.047; visual sphere radius=0.047
- link Head_upper: geometry collision cylinder length=0.09 radius=0.05; visual cylinder length=0.09 radius=0.05
