Commit message: add mimic gripper

File: source/robot_lab/data/Robots/go2_x5/go2_x5.urdf (robot description, URDF)
Before this commit: robot go2_x5, 52 links, 51 joints
Joints:
- joint arm_joint8: mimic (none) -> joint=arm_joint7 multiplier=1 offset=0

Commit message: Organize Go2-X5 docs and sim2sim workspace
Add public docs, script layout, sim2sim source/configs, UMI locomotion prototypes, and manipulation task scaffolds.

File: source/robot_lab/data/Robots/go2_x5/go2_x5.urdf (robot description, URDF)
Before this commit: robot go2_x5, 52 links, 51 joints
Links:
- link arm_base_link: mass 0.43995 -> 0.428; geometry visual mesh filename=./meshes/X5/base_link.STL
- link arm_link1: mass 0.066982 -> 0.064; geometry visual mesh filename=./meshes/X5/link1.STL
- link arm_link2: mass 1.0795 -> 1.165; geometry collision cylinder length=0.155 radius=0.025; visual mesh filename=./meshes/X5/link2.STL
- link arm_link3: mass 0.54534 -> 0.546; geometry collision cylinder length=0.15 radius=0.02; visual mesh filename=./meshes/X5/link3.STL
- link arm_link4: mass 0.11714 -> 0.100; geometry collision cylinder length=0.05 radius=0.025; visual mesh filename=./meshes/X5/link4.STL
- link arm_link5: mass 0.63488 -> 0.655; geometry visual mesh filename=./meshes/X5/link5.STL
- link arm_link6: mass 0.44089 -> 0.902; geometry collision box size=0.034 0.071 0.055; collision mesh filename=./meshes/X5/link6_truncated.stl
Joints:
- joint arm_base_joint: origin xyz=0.12 0 0.05 rpy=0 0 0 -> xyz=0.085 0 0.094 rpy=0 0 0
- joint arm_joint1: limit lower=-2.618 upper=3.14 effort=15 velocity=3 -> lower=-3.14159265359 upper=3.14159265359 effort=30 velocity=10; origin xyz=0 0 0.0605 rpy=0 0 0 -> xyz=0 0 0.0603 rpy=0 0 0
- joint arm_joint2: limit lower=0 upper=3.14 effort=15 velocity=3 -> lower=0 upper=3.66519 effort=30 velocity=10; origin xyz=0.02 0 0.04 rpy=0 0 0 -> xyz=0.02 0 0.0402 rpy=0 0 0
- joint arm_joint3: limit lower=0 upper=3.14 effort=15 velocity=3 -> lower=0 upper=3.14159265359 effort=30 velocity=10; origin xyz=-0.264 0 0 rpy=3.1416 0 0 -> xyz=-0.264 0 0 rpy=-3.1416 0 0
- joint arm_joint4: limit lower=-1.5708 upper=1.5708 effort=3 velocity=3 -> lower=-1.57079632679 upper=1.57079632679 effort=30 velocity=10
- joint arm_joint5: limit lower=-1.5708 upper=1.5708 effort=3 velocity=3 -> lower=-1.57079632679 upper=1.57079632679 effort=30 velocity=10; origin xyz=0.06775 0.0005 -0.0865 rpy=0 0 0 -> xyz=0.06575 -0.001 -0.0825 rpy=0 0 0
- joint arm_joint6: limit lower=-1.5708 upper=1.5708 effort=3 velocity=3 -> lower=-1.57079632679 upper=1.57079632679 effort=30 velocity=10; origin xyz=0.02895 0 0.0865 rpy=-3.1416 0 0 -> xyz=0.02845 0 0.0825 rpy=-3.1416 0 0
